File: hw/baybasi-ctrl.kicad_pcb (KiCad board)
At the start: 2 copper layers, 100 x 95 mm, 63 parts, among them J1 TerminalBlock_Phoenix_PT-1,5-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, J10 TerminalBlock_Phoenix_PT-1,5-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, J11 TerminalBlock_Phoenix_PT-1,5-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, J12 TerminalBlock_Phoenix_PT-1,5-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, J13 TerminalBlock_Phoenix_MKDS-1,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, J14 PinHeader_1x02_P2.54mm_Vertic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, J2 TerminalBlock_Phoenix_PT-1,5-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, J3 TerminalBlock_Phoenix_PT-1,5-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, J4 TerminalBlock_Phoenix_PT-1,5-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, J5 TerminalBlock_Phoenix_PT-1,5-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, J6 TerminalBlock_Phoenix_PT-1,5-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, J7 TerminalBlock_Phoenix_PT-1,5-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, J8 TerminalBlock_Phoenix_PT-1,5-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, J9 TerminalBlock_Phoenix_PT-1,5-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, M1 PinHeader_1x06_P2.54mm_Vertic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, M2 PinHeader_1x06_P2.54mm_Vertic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, Q1 SOT-23, U1 DIP-20_W7.62mm, U2 DIP-20_W7.62mm, U3 SOT-223-3_TabPin2

Commit message: hw: revB routed, DRC clean, gerbers exported
Board regenerated, routed and exported for the batch-2 run.

    0 DRC violations, 0 unconnected, 7 warnings
    all 7 are lib_footprint_mismatch - exactly batch 1's baseline

Getting there took three real fixes beyond the two intended changes:

**The right-hand cluster had to move with the socket.** A1R shifting 2.54 mm
right squeezed the A1R-to-U1 channel from ~7 mm to ~4.5 mm, and the router
could not keep the B.Cu pour continuous through it - isolated GND regions
around x 60-78, y 24-34. U1/U2 shifted +2.5 mm restores it. An earlier attempt
to paper over this with island_removal_mode made it worse (1 unconnected
region became 3) and is reverted; the channel was the cause, not the symptom.

**min_resolved_spokes is back to 1.** It went 1 -> 2 in commit 2cc4b0b, which
swept up an unvalidated working-tree change of mine and described it as "a DRC
tightening" without re-running DRC under it. It is the direct cause of 5
starved-thermal errors here (SW1 pads 7/8, A1R pad 1, J5/J8 pad 2). Batch 1
was fabricated and works at 1. Two spokes is a defensible standard but it
needs layout work, not a settings line.

**The silkscreen said revA.** Batch 2 would have shipped ten boards labelled
identically to the five already on the bench - except revA takes a 22.86 mm
devkit and revB takes 25.4 mm. Two boards that look the same, accept different
parts, and cannot be told apart without a caliper. Now split over two lines so
it clears SW1, with revB on its own line at full size.

Also adds the switch legend the spec asked for: pole weights 1 / 2 / SP / SP
beside their own poles, and COL=2+1 ON=1 below. Placing it cost three attempts
- the font runs ~0.74 mm per character at size 0.8, wider than I estimated
twice, and the board has very little free silkscreen area. The comments now
record the measured rate and say to check the placement box dump first.

CPL regenerated (U1/U2 moved, SW1 added). BOM carries SW1 / C99418.
Gerbers: baybasi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
Parts:
- added SW1: SW_DIP_SPSTx04_Slide_9.78x12.34mm_W7.62mm_P2.54mm, Button_Switch_THT:SW_DIP_SPSTx04_Slide_9.78x12.34mm_W7.62mm_P2.54mm, F.Cu at (124.0, 119.0)
- moved A1R 2.54 mm to (161.0, 67.0)
- moved U1 2.50 mm to (172.6, 66.5)
- moved U2 2.50 mm to (172.6, 96.5)
Connections:
- A1L pad 10: unconnected-(A1L-Pin_10-Pad10) -> COL_SP0
- A1L pad 11: unconnected-(A1L-Pin_11-Pad11) -> COL_SP1
- A1L pad 15: unconnected-(A1L-Pin_15-Pad15) -> COL_B0
- A1L pad 9: unconnected-(A1L-Pin_9-Pad9) -> COL_B1
Routing:
- net COL_SP0: track 0.00 -> 52.1 mm, vias 0 -> 2
- net COL_SP1: track 0.00 -> 49.2 mm, vias 0 -> 2
- net COL_B1: track 0.00 -> 45.1 mm
- net COL_B0: track 0.00 -> 22.6 mm, vias 0 -> 1
- net D8_5V: track 57.1 -> 72.7 mm
- net D3_3V3: track 56.1 -> 40.6 mm
- net D4_5V: track 44.5 -> 57.1 mm, vias 1 -> 2
- net OUT8: track 29.4 -> 41.1 mm, vias 1 -> 0
- net D7_5V: track 62.1 -> 72.2 mm, vias 0 -> 1
- net D6_5V: track 53.3 -> 44.3 mm, vias 2 -> 1
- net ETH_CS: track 43.4 -> 52.0 mm
- net +3V3E: track 144.8 -> 153.2 mm
- net OUT6: track 50.0 -> 55.6 mm, vias 3 -> 1
- net OUT4: track 38.6 -> 33.5 mm, vias 1 -> 0
- net D1_3V3: track 44.7 -> 39.9 mm
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Other:
- board text added: "1"
- board text added: "2"
- board text added: "BAYBASI COLUMN CTRL"
- board text added: "COL=2+1 ON=1"
- board text added: "SP"
- board text added: "revB"
- board text removed: "BAYBASI COLUMN CTRL revA"
